File: PCB/Guante/sensor_glove.brd (EAGLE design)
At the start: 56.8 x 56.8 mm, 43 parts, among them U1 MPU-6050, U2 STM32F030F4P6, U3 MCP73831, Y1 24MHz, Y2 16MHz

Commit message: Añadido interruptor en la PCB
Parts:
- added S3: (no value), SparkFun-Retired:SWITCH_SPDT_SMD
- moved J4 5.92 mm to (46.6, 23.9)
- moved J3 5.65 mm to (61.5, 24.5)
- moved C16 4.59 mm to (52.8, 27.2)
Connections:
- removed net N$30: C17.1, J4.2, U3.3
- new net CON: J4.2, S3.2
- net VCC: now also C17.1, S3.3, U3.3
Routing:
- net VCC: track 123.2 -> 146.9 mm, vias 10 -> 11
- net N$30: track 19.0 -> 0.00 mm
- net CON: track 0.00 -> 11.1 mm
- net GND: track 219.5 -> 223.1 mm
- net N$2: track 19.5 -> 16.6 mm
