File: PCB/Guante/sensor_glove.sch (EAGLE design)
At the start: 43 parts, among them U1 MPU-6050, U2 STM32F030F4P6, U3 MCP73831, Y1 24MHz, Y2 16MHz

Commit message: Añadido interruptor en la PCB
Parts:
- added S3: (no value), SparkFun-Retired:SWITCH-SPDTSMD
Connections:
- removed net N$30: C17.1, J4.+, U3.VBAT
- new net CON: J4.+, S3.P
- net VCC: now also C17.1, S3.S, U3.VBAT
Changed lines of the file:
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@@
 <part name="C5" library="SparkFun-Capacitors" deviceset="22PF" device="-0603-50V-5%" value="22pF"/>
 <part name="C6" library="SparkFun-Capacitors" deviceset="22PF" device="-0603-50V-5%" value="22pF"/>
+<part name="S3" library="SparkFun-Retired" deviceset="SWITCH-SPDT" device="SMD"/>
 </parts>
 <sheets>
@@
 <instance part="GND30" gate="1" x="182.88" y="38.1"/>
 <instance part="GND31" gate="1" x="193.04" y="55.88"/>
-<instance part="SUPPLY8" gate="G$1" x="205.74" y="55.88"/>
+<instance part="SUPPLY8" gate="G$1" x="220.98" y="55.88"/>
 <instance part="R12" gate="G$1" x="43.18" y="101.6"/>
 <instance part="C18" gate="G$1" x="-20.32" y="30.48" rot="R90"/>
@@
 <instance part="C5" gate="G$1" x="53.34" y="93.98"/>
 <instance part="C6" gate="G$1" x="35.56" y="93.98"/>
+<instance part="S3" gate="1" x="203.2" y="60.96" rot="R270"/>
 </instances>
 <busses>
@@
 <segment>
 <pinref part="SUPPLY8" gate="G$1" pin="VCC"/>
-<wire x1="205.74" y1="55.88" x2="205.74" y2="53.34" width="0.1524" layer="91"/>
+<wire x1="220.98" y1="55.88" x2="220.98" y2="53.34" width="0.1524" layer="91"/>
 </segment>
 <segment>
@@
 <wire x1="12.7" y1="73.66" x2="5.08" y2="73.66" width="0.1524" layer="91"/>
 <wire x1="5.08" y1="73.66" x2="5.08" y2="76.2" width="0.1524" layer="91"/>
+</segment>
+<segment>
+<pinref part="U3" gate="G$1" pin="VBAT"/>
+<wire x1="162.56" y1="53.34" x2="182.88" y2="53.34" width="0.1524" layer="91"/>
+<pinref part="C17" gate="G$1" pin="1"/>
+<wire x1="182.88" y1="53.34" x2="200.66" y2="53.34" width="0.1524" layer="91"/>
+<wire x1="200.66" y1="53.34" x2="220.98" y2="53.34" width="0.1524" layer="91"/>
+<wire x1="182.88" y1="53.34" x2="182.88" y2="50.8" width="0.1524" layer="91"/>
+<junction x="182.88" y="53.34"/>
+<pinref part="S3" gate="1" pin="S"/>
+<wire x1="200.66" y1="55.88" x2="200.66" y2="53.34" width="0.1524" layer="91"/>
+<junction x="200.66" y="53.34"/>
 </segment>
 </net>
@@
 </segment>
 </net>
-<net name="N$30" class="0">
-<segment>
-<pinref part="U3" gate="G$1" pin="VBAT"/>
-<wire x1="162.56" y1="53.34" x2="182.88" y2="53.34" width="0.1524" layer="91"/>
-<pinref part="C17" gate="G$1" pin="1"/>
-<wire x1="182.88" y1="53.34" x2="195.58" y2="53.34" width="0.1524" layer="91"/>
-<wire x1="195.58" y1="53.34" x2="205.74" y2="53.34" width="0.1524" layer="91"/>
-<wire x1="182.88" y1="53.34" x2="182.88" y2="50.8" width="0.1524" layer="91"/>
-<junction x="182.88" y="53.34"/>
+<net name="CON" class="0">
+<segment>
 <pinref part="J4" gate="G$1" pin="+"/>
-<wire x1="195.58" y1="66.04" x2="195.58" y2="53.34" width="0.1524" layer="91"/>
-<junction x="195.58" y="53.34"/>
-</segment>
-</net>
+<pinref part="S3" gate="1" pin="P"/>
+<wire x1="195.58" y1="66.04" x2="203.2" y2="66.04" width="0.1524" layer="91"/>
+<wire x1="203.2" y1="66.04" x2="203.2" y2="63.5" width="0.1524" layer="91"/>
+</segment>
+</net>
